File: Slave drones/Slave-Drone-backups/Slave-Drone-2026-06-07_181424/Slave-Drone.kicad_sch (KiCad schematic)
At the start: 41 parts, among them J1 Conn_01x02, J2 Conn_01x02, J3 Conn_01x02, J4 Conn_01x02, J5 USB_C_Receptacle_USB2.0_16P, J6 Conn_01x02, SW1 SW_Push, SW2 SW_Push, U1 MPU6500, U2 QMC5883L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

Commit message: I broke the pcb file, had to restart routing
Parts:
- U3: footprint ESP32-S3-MINI-1-N8:XCVR_ESP32-S3-MINI-1-N8 -> footprint-JLC:BULETM-SMD_ESP32-S3-MINI-1-N8
Connections:
- net +3.3V: now also U2.4 (S1)
Changed lines of the file:
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@@
 	)
 	(junction
+		(at 104.14 170.18)
+		(diameter 0)
+		(color 0 0 0 0)
+	)
+	(junction
 		(at 50.8 121.92)
 		(diameter 0)
@@
 	(wire
 		(pts
+			(xy 106.68 170.18) (xy 104.14 170.18)
+		)
+		(stroke
+			(width 0)
+			(type default)
+		)
+	)
+	(wire
+		(pts
 			(xy 236.22 124.46) (xy 236.22 125.73)
 		)
@@
 	(wire
 		(pts
+			(xy 104.14 165.1) (xy 104.14 170.18)
+		)
+		(stroke
+			(width 0)
+			(type default)
+		)
+	)
+	(wire
+		(pts
 			(xy 238.76 68.58) (xy 241.3 68.58)
 		)
@@
 	(wire
 		(pts
-			(xy 104.14 165.1) (xy 104.14 170.18)
-		)
-		(stroke
-			(width 0)
-			(type default)
-		)
-	)
-	(wire
-		(pts
 			(xy 63.5 29.21) (xy 72.39 29.21)
 		)
@@
 	(wire
 		(pts
+			(xy 104.14 170.18) (xy 95.25 170.18)
+		)
+		(stroke
+			(width 0)
+			(type default)
+		)
+	)
+	(wire
+		(pts
 			(xy 68.58 165.1) (xy 80.01 165.1)
 		)
@@
 	(wire
 		(pts
-			(xy 104.14 165.1) (xy 106.68 165.1)
-		)
-		(stroke
-			(width 0)
-			(type default)
-		)
-	)
-	(wire
-		(pts
 			(xy 213.36 121.92) (xy 213.36 125.73)
 		)
@@
 	(wire
 		(pts
-			(xy 95.25 170.18) (xy 104.14 170.18)
-		)
-		(stroke
-			(width 0)
-			(type default)
-		)
-	)
-	(wire
-		(pts
 			(xy 129.54 175.26) (xy 133.35 175.26)
 		)
@@
 	(wire
 		(pts
+			(xy 104.14 165.1) (xy 106.68 165.1)
+		)
+		(stroke
+			(width 0)
+			(type default)
+		)
+	)
+	(wire
+		(pts
 			(xy 259.08 66.04) (xy 242.57 66.04)
 		)
@@
 			)
 		)
-		(property "Footprint" "ESP32-S3-MINI-1-N8:XCVR_ESP32-S3-MINI-1-N8"
+		(property "Footprint" "footprint-JLC:BULETM-SMD_ESP32-S3-MINI-1-N8"
 			(at 167.64 119.38 0)
 			(hide yes)
